File: 4CHLED/4ch_lpc.sch (EAGLE design)
At the start: 52 parts, among them IC1 LT1761, IC2 MAX487CSA, IC3 LT3972, IC4 78L05SMD, Q1 MT-OSCILLATOR, T1 IRF7103, T2 IRF7103, X1 RJ45-8L-B, X2 RJ45-8L-B, X4 87758-0616

Commit message: final touches for production
Parts:
- added R17: 68k, SparkFun:RESISTOR0402-RES
- renumbered U1 to IC5
Connections:
- net !RE: now also R17.2
- net +3V3: now also IC5.PIO0_3
- net GND: now also R17.1
Changed lines of the file:
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@@
 <part name="SUPPLY1" library="supply2" deviceset="+4.1V" device=""/>
 <part name="SUPPLY2" library="supply2" deviceset="+4.1V" device=""/>
-<part name="U1" library="microbuilder" deviceset="LPC1113/4_QFN" device=""/>
+<part name="IC5" library="microbuilder" deviceset="LPC1113/4_QFN" device=""/>
 <part name="GND1" library="supply1" deviceset="GND" device=""/>
 <part name="P+1" library="supply1" deviceset="+5V" device=""/>
@@
 <part name="GND11" library="supply1" deviceset="GND" device=""/>
 <part name="P+4" library="supply1" deviceset="+5V" device=""/>
+<part name="R17" library="SparkFun" deviceset="RESISTOR" device="0402-RES" value="68k"/>
+<part name="GND12" library="supply1" deviceset="GND" device=""/>
+<part name="+3V6" library="supply1" deviceset="+3V3" device=""/>
 </parts>
 <sheets>
@@
 <instance part="SUPPLY1" gate="P" x="383.54" y="129.54"/>
 <instance part="SUPPLY2" gate="P" x="86.36" y="15.24" rot="R90"/>
-<instance part="U1" gate="G$1" x="195.58" y="45.72"/>
+<instance part="IC5" gate="G$1" x="195.58" y="45.72"/>
 <instance part="GND1" gate="1" x="124.46" y="22.86" rot="R270"/>
 <instance part="P+1" gate="1" x="149.86" y="147.32"/>
@@
 <instance part="GND11" gate="1" x="129.54" y="-12.7" rot="R270"/>
 <instance part="P+4" gate="1" x="129.54" y="-15.24" rot="R90"/>
+<instance part="R17" gate="G$1" x="33.02" y="127" rot="R90"/>
+<instance part="GND12" gate="1" x="33.02" y="119.38"/>
+<instance part="+3V6" gate="G$1" x="132.08" y="60.96" rot="R90"/>
 </instances>
 <busses>
@@
 <segment>
 <pinref part="GND1" gate="1" pin="GND"/>
-<pinref part="U1" gate="G$1" pin="VSS"/>
+<pinref part="IC5" gate="G$1" pin="VSS"/>
 <wire x1="127" y1="22.86" x2="144.78" y2="22.86" width="0.1524" layer="91"/>
 </segment>
@@
 <pinref part="GND11" gate="1" pin="GND"/>
 </segment>
+<segment>
+<pinref part="R17" gate="G$1" pin="1"/>
+<pinref part="GND12" gate="1" pin="GND"/>
+</segment>
 </net>
 <net name="+5V" class="0">
@@
 </segment>
 <segment>
-<pinref part="U1" gate="G$1" pin="PIO1_7/TXD/CT32B0_MAT1"/>
+<pinref part="IC5" gate="G$1" pin="PIO1_7/TXD/CT32B0_MAT1"/>
 <wire x1="248.92" y1="50.8" x2="264.16" y2="50.8" width="0.1524" layer="91"/>
 <label x="259.08" y="50.8" size="1.778" layer="95"/>
@@
 </segment>
 <segment>
-<pinref part="U1" gate="G$1" pin="PIO1_6/RXD/CT32B0_MAT0"/>
+<pinref part="IC5" gate="G$1" pin="PIO1_6/RXD/CT32B0_MAT0"/>
 <wire x1="248.92" y1="53.34" x2="264.16" y2="53.34" width="0.1524" layer="91"/>
 <label x="259.08" y="53.34" size="1.778" layer="95"/>
@@
 <net name="!RE" class="0">
 <segment>
-<wire x1="48.26" y1="134.62" x2="40.64" y2="134.62" width="0.1524" layer="91"/>
 <wire x1="48.26" y1="134.62" x2="48.26" y2="129.54" width="0.1524" layer="91"/>
 <junction x="48.26" y="134.62"/>
@@
 <pinref part="IC2" gate="G$1" pin="RE/"/>
 <pinref part="IC2" gate="G$1" pin="DE"/>
-</segment>
-<segment>
-<pinref part="U1" gate="G$1" pin="PIO1_5/RTS/CT32B0_CAP0"/>
+<pinref part="R17" gate="G$1" pin="2"/>
+<wire x1="48.26" y1="134.62" x2="33.02" y2="134.62" width="0.1524" layer="91"/>
+<wire x1="33.02" y1="134.62" x2="33.02" y2="132.08" width="0.1524" layer="91"/>
+</segment>
+<segment>
+<pinref part="IC5" gate="G$1" pin="PIO1_5/RTS/CT32B0_CAP0"/>
 <wire x1="248.92" y1="55.88" x2="264.16" y2="55.88" width="0.1524" layer="91"/>
 <label x="259.08" y="55.88" size="1.778" layer="95"/>
@@
 </segment>
 <segment>
-<pinref part="U1" gate="G$1" pin="TRST/PIO1_2/AD3/CT32B1_MAT1"/>
+<pinref part="IC5" gate="G$1" pin="TRST/PIO1_2/AD3/CT32B1_MAT1"/>
 <wire x1="248.92" y1="63.5" x2="264.16" y2="63.5" width="0.1524" layer="91"/>
 <label x="259.08" y="63.5" size="1.778" layer="95"/>
@@
 </segment>
 <segment>
-<pinref part="U1" gate="G$1" pin="SWDIO/PIO1_3/AD4/CT32B1_MAT2"/>
+<pinref part="IC5" gate="G$1" pin="SWDIO/PIO1_3/AD4/CT32B1_MAT2"/>
 <wire x1="248.92" y1="60.96" x2="264.16" y2="60.96" width="0.1524" layer="91"/>
 <label x="259.08" y="60.96" size="1.778" layer="95"/>
@@
 </segment>
 <segment>
-<pinref part="U1" gate="G$1" pin="PIO1_4/AD5/CT32B1_MAT3/WAKEUP"/>
+<pinref part="IC5" gate="G$1" pin="PIO1_4/AD5/CT32B1_MAT3/WAKEUP"/>
 <wire x1="248.92" y1="58.42" x2="264.16" y2="58.42" width="0.1524" layer="91"/>
 <label x="259.08" y="58.42" size="1.778" layer="95"/>
@@
 </segment>
 <segment>
-<pinref part="U1" gate="G$1" pin="TDO/PIO1_1/AD2/CT32B1_MAT0"/>
+<pinref part="IC5" gate="G$1" pin="TDO/PIO1_1/AD2/CT32B1_MAT0"/>
 <wire x1="248.92" y1="66.04" x2="264.16" y2="66.04" width="0.1524" layer="91"/>
 <label x="259.08" y="66.04" size="1.778" layer="95"/>
@@
 <wire x1="271.78" y1="71.12" x2="274.32" y2="71.12" width="0.1524" layer="91"/>
 <wire x1="274.32" y1="71.12" x2="274.32" y2="27.94" width="0.1524" layer="91"/>
-<pinref part="U1" gate="G$1" pin="PIO3_4"/>
+<pinref part="IC5" gate="G$1" pin="PIO3_4"/>
 <wire x1="274.32" y1="27.94" x2="248.92" y2="27.94" width="0.1524" layer="91"/>
 </segment>
@@
 </segment>
 <segment>
-<pinref part="U1" gate="G$1" pin="VDD(IO)"/>
+<pinref part="IC5" gate="G$1" pin="VDD(IO)"/>
 <pinref part="+3V2" gate="G$1" pin="+3V3"/>
 <wire x1="144.78" y1="25.4" x2="129.54" y2="25.4" width="0.1524" layer="91"/>
 <wire x1="129.54" y1="25.4" x2="129.54" y2="27.94" width="0.1524" layer="91"/>
-<pinref part="U1" gate="G$1" pin="VDD(3V3)"/>
+<pinref part="IC5" gate="G$1" pin="VDD(3V3)"/>
 <wire x1="129.54" y1="27.94" x2="129.54" y2="30.48" width="0.1524" layer="91"/>
 <wire x1="144.78" y1="27.94" x2="129.54" y2="27.94" width="0.1524" layer="91"/>
@@
 <pinref part="+3V5" gate="G$1" pin="+3V3"/>
 </segment>
+<segment>
+<pinref part="+3V6" gate="G$1" pin="+3V3"/>
+<pinref part="IC5" gate="G$1" pin="PIO0_3"/>
+<wire x1="134.62" y1="60.96" x2="144.78" y2="60.96" width="0.1524" layer="91"/>
+</segment>
 </net>
 <net name="N$7" class="0">
@@
 <net name="RST" class="0">
 <segment>
-<pinref part="U1" gate="G$1" pin="RESET/PIO0_0"/>
+<pinref part="IC5" gate="G$1" pin="RESET/PIO0_0"/>
 <wire x1="144.78" y1="68.58" x2="132.08" y2="68.58" width="0.1524" layer="91"/>
 <pinref part="R1" gate="G$1" pin="2"/>
@@
 <net name="BL" class="0">
 <segment>
-<pinref part="U1" gate="G$1" pin="PIO0_1/CLKOUT/CT32B0_MAT2"/>
+<pinref part="IC5" gate="G$1" pin="PIO0_1/CLKOUT/CT32B0_MAT2"/>
 <wire x1="144.78" y1="66.04" x2="137.16" y2="66.04" width="0.1524" layer="91"/>
 <pinref part="R16" gate="G$1" pin="2"/>
@@
 <wire x1="119.38" y1="40.64" x2="134.62" y2="40.64" width="0.1524" layer="91"/>
 <wire x1="134.62" y1="40.64" x2="134.62" y2="33.02" width="0.1524" layer="91"/>
-<pinref part="U1" gate="G$1" pin="XTALOUT"/>
+<pinref part="IC5" gate="G$1" pin="XTALOUT"/>
 <wire x1="134.62" y1="33.02" x2="144.78" y2="33.02" width="0.1524" layer="91"/>
 <pinref part="C5" gate="G$1" pin="2"/>
@@
 <net name="N$21" class="0">
 <segment>
-<pinref part="U1" gate="G$1" pin="XTALIN"/>
+<pinref part="IC5" gate="G$1" pin="XTALIN"/>
 <wire x1="144.78" y1="35.56" x2="137.16" y2="35.56" width="0.1524" layer="91"/>
 <wire x1="137.16" y1="35.56" x2="137.16" y2="45.72" width="0.1524" layer="91"/>
